Commit message: collision checkiing safeties for S2R

File: skillet_tasks/assets/kortex/kinova_gen3/gen3_2f85.urdf (robot description, URDF)
Before this commit: robot gen3_, 32 links, 31 joints
Links:
- link gen3_base_link: geometry collision mesh filename=meshes/base_link.dae; visual mesh filename=meshes/base_link.dae
- link gen3_bracelet_link: geometry collision mesh filename=meshes/bracelet_no_vision_link.dae; visual mesh filename=meshes/bracelet_no_vision_link.dae
- link gen3_forearm_link: geometry collision mesh filename=meshes/forearm_link.dae; visual mesh filename=meshes/forearm_link.dae
- link gen3_half_arm_1_link: geometry collision mesh filename=meshes/half_arm_1_link.dae; visual mesh filename=meshes/half_arm_1_link.dae
- link gen3_half_arm_2_link: geometry collision mesh filename=meshes/half_arm_2_link.dae; visual mesh filename=meshes/half_arm_2_link.dae
- link gen3_robotiq_85_base_link: geometry collision mesh filename=meshes/robotiq_base.stl; visual mesh filename=meshes/robotiq_base.dae
- link gen3_robotiq_85_left_finger_link: geometry collision mesh filename=meshes/left_finger.stl; visual mesh filename=meshes/left_finger.dae
- link gen3_robotiq_85_left_finger_tip_link: geometry collision mesh filename=meshes/left_finger_tip.stl; visual mesh filename=meshes/left_finger_tip.dae
- link gen3_robotiq_85_left_inner_knuckle_link: geometry collision mesh filename=meshes/left_inner_knuckle.stl; visual mesh filename=meshes/left_inner_knuckle.dae
- link gen3_robotiq_85_left_knuckle_link: geometry collision mesh filename=meshes/left_knuckle.stl; visual mesh filename=meshes/left_knuckle.dae
- link gen3_robotiq_85_right_finger_link: geometry collision mesh filename=meshes/right_finger.stl; visual mesh filename=meshes/right_finger.dae
- link gen3_robotiq_85_right_finger_tip_link: geometry collision mesh filename=meshes/right_finger_tip.stl; visual mesh filename=meshes/right_finger_tip.dae
- link gen3_robotiq_85_right_inner_knuckle_link: geometry collision mesh filename=meshes/right_inner_knuckle.stl; visual mesh filename=meshes/right_inner_knuckle.dae
- link gen3_robotiq_85_right_knuckle_link: geometry collision mesh filename=meshes/right_knuckle.stl; visual mesh filename=meshes/right_knuckle.dae
- link gen3_shoulder_link: geometry collision mesh filename=meshes/shoulder_link.dae; visual mesh filename=meshes/shoulder_link.dae
- link gen3_spherical_wrist_1_link: geometry collision mesh filename=meshes/spherical_wrist_1_link.dae; visual mesh filename=meshes/spherical_wrist_1_link.dae
- link gen3_spherical_wrist_2_link: geometry collision mesh filename=meshes/spherical_wrist_2_link.dae; visual mesh filename=meshes/spherical_wrist_2_link.dae
- link wrist_camera_mount_link: geometry collision mesh filename=meshes//realsense_bracket_for_kinova.dae; visual mesh filename=meshes/realsense_bracket_for_kinova.dae

File: skillet_tasks/assets/kortex/kinova_gen3lite/gen3_lite.urdf (robot description, URDF)
Before this commit: robot gen3_lite, 15 links, 14 joints
Links:
- link arm_link: geometry collision mesh filename=meshes/arm_link.STL; visual mesh filename=meshes/arm_link.STL
- link base_link: geometry collision mesh filename=meshes/base_link.STL; visual mesh filename=meshes/base_link.STL
- link forearm_link: geometry collision mesh filename=meshes/forearm_link.STL; visual mesh filename=meshes/forearm_link.STL
- link gripper_base_link: geometry collision mesh filename=meshes/gripper_base_link.STL; visual mesh filename=meshes/gripper_base_link.STL
- link left_finger_dist_link: geometry collision mesh filename=meshes/left_finger_dist_link.STL; visual mesh filename=meshes/left_finger_dist_link.STL
- link left_finger_prox_link: geometry collision mesh filename=meshes/left_finger_prox_link.STL; visual mesh filename=meshes/left_finger_prox_link.STL
- link lower_wrist_link: geometry collision mesh filename=meshes/lower_wrist_link.STL; visual mesh filename=meshes/lower_wrist_link.STL
- link right_finger_dist_link: geometry collision mesh filename=meshes/right_finger_dist_link.STL; visual mesh filename=meshes/right_finger_dist_link.STL
- link right_finger_prox_link: geometry collision mesh filename=meshes/right_finger_prox_link.STL; visual mesh filename=meshes/right_finger_prox_link.STL
- link shoulder_link: geometry collision mesh filename=meshes/shoulder_link.STL; visual mesh filename=meshes/shoulder_link.STL
- link upper_wrist_link: geometry collision mesh filename=meshes/upper_wrist_link.STL; visual mesh filename=meshes/upper_wrist_link.STL

Commit message: initial changes to gen3.. not working currently

File: skillet_tasks/assets/kortex/kinova_gen3/gen3_2f85.urdf (robot description, URDF)
Before this commit: robot gen3_, 32 links, 31 joints
Links:
- removed link gen3_base_link
- removed link gen3_bracelet_link
- removed link gen3_end_effector_link
- removed link gen3_forearm_link
- removed link gen3_half_arm_1_link
- removed link gen3_half_arm_2_link
- removed link gen3_robotiq_85_base_link
- removed link gen3_robotiq_85_left_finger_link
- removed link gen3_robotiq_85_left_finger_tip_link
- removed link gen3_robotiq_85_left_inner_knuckle_link
- removed link gen3_robotiq_85_left_knuckle_link
- removed link gen3_robotiq_85_right_finger_link
- removed link gen3_robotiq_85_right_finger_tip_link
- removed link gen3_robotiq_85_right_inner_knuckle_link
- removed link gen3_robotiq_85_right_knuckle_link
- removed link gen3_shoulder_link
- removed link gen3_spherical_wrist_1_link
- removed link gen3_spherical_wrist_2_link
- removed link gen3_tool_frame
- added link base_link, mass 1.697; collision mesh filename=meshes/base_link.dae; visual mesh filename=meshes/base_link.dae
- added link bracelet_link, mass 0.364; collision mesh filename=meshes/bracelet_no_vision_link.dae; visual mesh filename=meshes/bracelet_no_vision_link.dae
- added link end_effector_link
- added link forearm_link, mass 0.9302; collision mesh filename=meshes/forearm_link.dae; visual mesh filename=meshes/forearm_link.dae
- added link half_arm_1_link, mass 1.1636; collision mesh filename=meshes/half_arm_1_link.dae; visual mesh filename=meshes/half_arm_1_link.dae
- added link half_arm_2_link, mass 1.1636; collision mesh filename=meshes/half_arm_2_link.dae; visual mesh filename=meshes/half_arm_2_link.dae
- added link robotiq_85_base_link, mass 6.6320197e-01; collision mesh filename=meshes/robotiq_base.stl; visual mesh filename=meshes/robotiq_base.dae
- added link robotiq_85_left_finger_link, mass 4.260376752e-02; collision mesh filename=meshes/left_finger.stl; visual mesh filename=meshes/left_finger.dae
- added link robotiq_85_left_finger_tip_link, mass 4.268588744e-02; collision mesh filename=meshes/left_finger_tip.stl; visual mesh filename=meshes/left_finger_tip.dae
- added link robotiq_85_left_inner_knuckle_link, mass 2.969376448e-02; collision mesh filename=meshes/left_inner_knuckle.stl; visual mesh filename=meshes/left_inner_knuckle.dae
- added link robotiq_85_left_knuckle_link, mass 1.384773208e-02; collision mesh filename=meshes/left_knuckle.stl; visual mesh filename=meshes/left_knuckle.dae
- added link robotiq_85_right_finger_link, mass 4.260376752000000e-02; collision mesh filename=meshes/right_finger.stl; visual mesh filename=meshes/right_finger.dae
- added link robotiq_85_right_finger_tip_link, mass 4.268588744e-02; collision mesh filename=meshes/right_finger_tip.stl; visual mesh filename=meshes/right_finger_tip.dae
- added link robotiq_85_right_inner_knuckle_link, mass 2.969376448e-02; collision mesh filename=meshes/right_inner_knuckle.stl; visual mesh filename=meshes/right_inner_knuckle.dae
- added link robotiq_85_right_knuckle_link, mass 1.384773208e-02; collision mesh filename=meshes/right_knuckle.stl; visual mesh filename=meshes/right_knuckle.dae
- added link shoulder_link, mass 1.3773; collision mesh filename=meshes/shoulder_link.dae; visual mesh filename=meshes/shoulder_link.dae
- added link spherical_wrist_1_link, mass 0.6781; collision mesh filename=meshes/spherical_wrist_1_link.dae; visual mesh filename=meshes/spherical_wrist_1_link.dae
- added link spherical_wrist_2_link, mass 0.6781; collision mesh filename=meshes/spherical_wrist_2_link.dae; visual mesh filename=meshes/spherical_wrist_2_link.dae
- link wrist_camera_mount_link: geometry 
- link wrist_mounted_camera_link: geometry collision box size=0.02005 0.099 0.023; visual mesh filename=meshes/d415.stl
Joints:
- removed joint gen3_base_joint
- removed joint gen3_end_effector
- removed joint gen3_joint_1
- removed joint gen3_joint_2
- removed joint gen3_joint_3
- removed joint gen3_joint_4
- removed joint gen3_joint_5
- removed joint gen3_joint_6
- removed joint gen3_joint_7
- removed joint gen3_robotiq_85_base_joint
- removed joint gen3_robotiq_85_left_finger_joint
- removed joint gen3_robotiq_85_left_finger_tip_joint
- removed joint gen3_robotiq_85_left_inner_knuckle_joint
- removed joint gen3_robotiq_85_left_knuckle_joint
- removed joint gen3_robotiq_85_right_finger_joint
- removed joint gen3_robotiq_85_right_finger_tip_joint
- removed joint gen3_robotiq_85_right_inner_knuckle_joint
- removed joint gen3_robotiq_85_right_knuckle_joint
- removed joint gen3_tool_frame_joint
- added joint base_joint: type fixed, parent world, child base_link, origin xyz=0 0 0 rpy=0 0 0
- added joint end_effector: type fixed, parent bracelet_link, child end_effector_link, origin xyz=0 0 -0.0615250000000001 rpy=3.14159265358979 1.09937075168372E-32 0, axis 0 0 0
- added joint joint_1: type continuous, parent base_link, child shoulder_link, origin xyz=0 0 0.15643 rpy=3.1416 2.7629E-18 -4.9305E-36, axis 0 0 1, limit effort=39 velocity=1.3963
- added joint joint_2: type revolute, parent shoulder_link, child half_arm_1_link, origin xyz=0 0.005375 -0.12838 rpy=1.5708 2.1343E-17 -1.1102E-16, axis 0 0 1, limit lower=-2.41 upper=2.41 effort=39 velocity=1.3963
- added joint joint_3: type continuous, parent half_arm_1_link, child half_arm_2_link, origin xyz=0 -0.21038 -0.006375 rpy=-1.5708 1.2326E-32 -2.9122E-16, axis 0 0 1, limit effort=39 velocity=1.3963
- added joint joint_4: type revolute, parent half_arm_2_link, child forearm_link, origin xyz=0 0.006375 -0.21038 rpy=1.5708 -6.6954E-17 -1.6653E-16, axis 0 0 1, limit lower=-2.66 upper=2.66 effort=39 velocity=1.3963
- added joint joint_5: type continuous, parent forearm_link, child spherical_wrist_1_link, origin xyz=0 -0.20843 -0.006375 rpy=-1.5708 2.2204E-16 -6.373E-17, axis 0 0 1, limit effort=9 velocity=1.2218
- added joint joint_6: type revolute, parent spherical_wrist_1_link, child spherical_wrist_2_link, origin xyz=0 0.00017505 -0.10593 rpy=1.5708 9.2076E-28 -8.2157E-15, axis 0 0 1, limit lower=-2.23 upper=2.23 effort=9 velocity=1.2218
- added joint joint_7: type continuous, parent spherical_wrist_2_link, child bracelet_link, origin xyz=0 -0.10593 -0.00017505 rpy=-1.5708 -5.5511E-17 9.6396E-17, axis 0 0 1, limit effort=9 velocity=1.2218
- added joint robotiq_85_base_joint: type fixed, parent end_effector_link, child robotiq_85_base_link, origin xyz=0 0 0 rpy=0 0 0
- added joint robotiq_85_left_finger_joint: type fixed, parent robotiq_85_left_knuckle_link, child robotiq_85_left_finger_link, origin xyz=0.03152616 0.0 -0.00376347 rpy=0 0 0
- added joint robotiq_85_left_finger_tip_joint: type continuous, parent robotiq_85_left_finger_link, child robotiq_85_left_finger_tip_link, origin xyz=0.00563134 0.0 0.04718515 rpy=0 0 0, axis 0 -1 0, mimic joint=robotiq_85_left_knuckle_joint multiplier=-1
- added joint robotiq_85_left_inner_knuckle_joint: type continuous, parent robotiq_85_base_link, child robotiq_85_left_inner_knuckle_link, origin xyz=0.0127 0.0 0.06142 rpy=0 0 0, axis 0 -1 0, mimic joint=robotiq_85_left_knuckle_joint
- added joint robotiq_85_left_knuckle_joint: type revolute, parent robotiq_85_base_link, child robotiq_85_left_knuckle_link, origin xyz=0.03060114 0.0 0.05490452 rpy=0 0 0, axis 0 -1 0, limit lower=0.0 upper=0.8 effort=50 velocity=0.5
- added joint robotiq_85_right_finger_joint: type fixed, parent robotiq_85_right_knuckle_link, child robotiq_85_right_finger_link, origin xyz=-0.03152616 0.0 -0.00376347 rpy=0 0 0
- added joint robotiq_85_right_finger_tip_joint: type continuous, parent robotiq_85_right_finger_link, child robotiq_85_right_finger_tip_link, origin xyz=-0.00563134 0.0 0.04718515 rpy=0 0 0, axis 0 -1 0, mimic joint=robotiq_85_left_knuckle_joint
- added joint robotiq_85_right_inner_knuckle_joint: type continuous, parent robotiq_85_base_link, child robotiq_85_right_inner_knuckle_link, origin xyz=-0.0127 0.0 0.06142 rpy=0 0 0, axis 0 -1 0, mimic joint=robotiq_85_left_knuckle_joint multiplier=-1
- added joint robotiq_85_right_knuckle_joint: type revolute, parent robotiq_85_base_link, child robotiq_85_right_knuckle_link, origin xyz=-0.03060114 0.0 0.05490452 rpy=0 0 0, axis 0 -1 0, limit lower=-0.8 upper=0.0 effort=50 velocity=0.5, mimic joint=robotiq_85_left_knuckle_joint multiplier=-1
- joint wrist_camera_joint: parent gen3_bracelet_link -> bracelet_link
- joint wrist_camera_mount_joint: parent gen3_bracelet_link -> bracelet_link
